Commit message: [feat]:灯模块修改以及说明

File: src/aquaflow_stonefish/model/robot/bluerov2.urdf (robot description, URDF)
Before this commit: robot multipleshapes, 1 links, 0 joints
Links:
- link base_link: geometry visual mesh filename=package://aquaflow_stonefish/model/robot/bluerov2/bluerov2.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 scale=1.0 1.0 1.0

File: src/aquaflow_stonefish/model/robot/bricsbot/bricsbot.urdf (robot description, URDF)
Before this commit: robot bricsbot, 3 links, 2 joints
Links:
- link base_link: geometry visual mesh filename=package://aquaflow_stonefish/model/robot/bricsbot/bot_shark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 scale=1 1 1
